File: rp2040-promicro/rp2040-promicro.kicad_sch (KiCad schematic)
At the start: 30 parts, among them J2 ProMicro-LeftPin, J3 ProMicro-RightPin, P1 USB2.0_C_12pin, SW1 SW_Push, U1 RP2040, U2 W25Q128JVS, U3 AZ1117-3.3, Y1 Crystal_GND24

Commit message: promicro v2
Parts:
- removed C4: 100nF, rp2040-dev-board:Capacitor_0805_2012, symbol Device:C
- removed J2: ProMicro-LeftPin, rp2040-dev-board:LeftPin, symbol rp2040-dev-board:ProMicro-LeftPin
- removed J3: ProMicro-RightPin, rp2040-dev-board:RightPin, symbol rp2040-dev-board:ProMicro-RightPin
- removed P1: USB2.0_C_12pin, rp2040-dev-board:USB-C-12-Pin-MidMount-ali-v2, symbol rp2040-dev-board:USB2.0_C_12pin
- added F1: Polyfuse, $74th:ResettableFuse_KT6-1100SMDI, symbol Device:Polyfuse
- added J1: USB2.0_C_v3, $74th:USB-C-12-Pin-SMD, symbol $74th:USB2.0_C_v3
- added J2: ProMicro-LeftPin, $74th:ProMicro_LIKE_LEFT, symbol $74th:ProMicro-LeftPin
- added J3: ProMicro-RightPin, $74th:ProMicro_LIKE_RIGHT, symbol $74th:ProMicro-RightPin
- added R8: 1kR, rp2040-dev-board:Register_0805_2012, symbol Device:R
- C11, C12: footprint rp2040-dev-board:Capacitor_0603_1608 -> rp2040-dev-board:Capacitor_0805_2012
- SW1: footprint rp2040-dev-board:BOOT -> rp2040-dev-board:SKRPABE010
- U3: footprint rp2040-dev-board:Regulator-AMS1117-SOT-223 -> $74th:Regulator_AMS1117_SOT-89
- Y1: footprint Crystal:Crystal_SMD_3225-4Pin_3.2x2.5mm_HandSoldering -> rp2040-dev-board:Crystal_SMD_3225-4Pin_3.2x2.5mm_HandSoldering
Connections:
- net +3V3: now also J3.9 (3V3)
- net +5V: now also F1.2, J3.12 (RAW)
- net 0/TX0: now also J2.1 (1/TX)
- net 1/RX0: now also J2.2 (0/RX)
- net 2: now also J2.5 (2/SDA)
- net 20: now also J3.3 (14/SPI_MISO)
- net 21: now also J3.1 (10/A10)
- net 22: now also J3.4 (15/SPI_SCK)
- net 23: now also J3.2 (16/SPI_MOSI)
- net 3: now also J2.6 (3/SCL)
- net 4: now also J2.7 (4/A6)
- net 5: now also J2.8 (5)
- net 6: now also J2.9 (6/A7)
- net 7: now also J2.10 (7)
- net 8/TX1: now also J2.11 (8/A8)
- net 9/RX1: now also J2.12 (9/A9)
- net A0: now also J3.5 (18/A0)
- net A1: now also J3.6 (19/A1)
- net A2: now also J3.7 (20/A2)
- net A3: now also J3.8 (21/A3)
- net GND: now also J1.4 (GND), J2.3 (GND), J2.4 (GND), J3.11 (GND)
- net USB_DM: now also J1.2 (D-)
- net USB_DP: now also J1.3 (D+)
- net XOUT: now also R8.1; no longer C12.2, Y1.3
- net ~{RESET}: now also J3.10 (~{RESET})
- net at R5.1: now also J1.5 (CC1)
- net at R4.1: now also J1.6 (CC2)
- new net: C12.2, R8.2, Y1.3
- new net: F1.1, J1.1 (VBUS)
- no-connect marks 16 -> 14
Other:
- title: (none) -> RP-ProMicro
- moved on the sheet: C14, C15, R1, R2, R4, R5, U3

Commit message: rp-promicro v2.0.0
Parts:
- U1: MPN (none) -> C2040
- U2: footprint rp2040-dev-board:W25Q16-128JV-SOIC -> Package_SO:SOIC-8_5.23x5.23mm_P1.27mm
Changed lines of the file:
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@@
       (effects (font (size 1.27 1.27)) (justify left))
     )
-    (property "Footprint" "rp2040-dev-board:W25Q16-128JV-SOIC" (id 2) (at 199.39 91.44 0)
+    (property "Footprint" "Package_SO:SOIC-8_5.23x5.23mm_P1.27mm" (id 2) (at 199.39 91.44 0)
       (effects (font (size 1.27 1.27)) hide)
     )
@@
       (effects (font (size 1.27 1.27)) hide)
     )
+    (property "MPN" "C2040" (id 4) (at 63.5 115.57 0))
     (pin "1")
     (pin "10")
@@
     )
     (path "/3adb8733-e6c3-4881-a255-9c7f78952e3e"
-      (reference "U2") (unit 1) (value "W25Q128JVS") (footprint "rp2040-dev-board:W25Q16-128JV-SOIC")
+      (reference "U2") (unit 1) (value "W25Q128JVS") (footprint "Package_SO:SOIC-8_5.23x5.23mm_P1.27mm")
     )
     (path "/a42a968a-2172-48a4-b850-dbe3a7175592"

Commit message: rp-promicro v2.0.0
Parts:
- U2: footprint Package_SO:SOIC-8_5.23x5.23mm_P1.27mm -> $74th:W25Q16-128JV-SOIC
Changed lines of the file:
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@@
       (effects (font (size 1.27 1.27)) (justify left))
     )
-    (property "Footprint" "Package_SO:SOIC-8_5.23x5.23mm_P1.27mm" (id 2) (at 199.39 91.44 0)
+    (property "Footprint" "$74th:W25Q16-128JV-SOIC" (id 2) (at 199.39 91.44 0)
       (effects (font (size 1.27 1.27)) hide)
     )
@@
     )
     (path "/3adb8733-e6c3-4881-a255-9c7f78952e3e"
-      (reference "U2") (unit 1) (value "W25Q128JVS") (footprint "Package_SO:SOIC-8_5.23x5.23mm_P1.27mm")
+      (reference "U2") (unit 1) (value "W25Q128JVS") (footprint "$74th:W25Q16-128JV-SOIC")
     )
     (path "/a42a968a-2172-48a4-b850-dbe3a7175592"
