File: rp2040-large/rp2040-large.kicad_pcb (KiCad board)
At the start: 2 copper layers, 21.3 x 51.6 mm, 30 parts, among them P1 USB2.0_C_12pin, P2 20Pin, P3 20Pin, SW1 SW_Push, U1 RP2040, U2 W25Q128JVS, U3 AZ1117-3.3, Y1 Crystal_GND24

Commit message: rp2040-large v1.4.0
Parts:
- removed P1: USB2.0_C_12pin, rp2040-dev-board:USB-C-12-Pin-MidMount-ali-v2
- added C16: 100nF, rp2040-dev-board:Capacitor_0805_2012, B.Cu at (116.1, 74.4)
- added J1: USB2.0_C_v3, rp2040-dev-board:USB-C-12-Pin-MidMount-ali-v4, F.Cu at (118.1, 38.9)
- added J2: SWD, rp2040-dev-board:SWD_PIN, F.Cu at (124.5, 78.7)
- added R10: 1R, rp2040-dev-board:Register_0805_2012, B.Cu at (122.7, 46.5)
- added R8: 10kR, rp2040-dev-board:Register_0805_2012, B.Cu at (112.8, 52.0)
- added R9: 200R, rp2040-dev-board:Register_0805_2012, B.Cu at (121.7, 43.2)
- added SW2: SW_Push, rp2040-dev-board:SKRPABE010, F.Cu at (124.0, 51.2)
- C1, C10, C13, C15, C2, C3, C4, C5, C6, C7, C8, R1, R2, R3, R4, R5, R7: moved to B.Cu
- C11, C12: footprint rp2040-dev-board:Capacitor_0603_1608 -> rp2040-dev-board:Capacitor_0805_2012
- C9: value 100nF -> 1uF; moved to B.Cu
- R6: value 10kR -> 1kR
- SW1: footprint rp2040-dev-board:2Pin -> rp2040-dev-board:SKRPABE010
- moved R6 28.9 mm to (118.0, 76.7)
- moved C3 16.5 mm to (121.2, 61.0), turned to 90 degrees
- moved C5 16.5 mm to (116.2, 64.1)
- moved C10 15.7 mm to (113.0, 71.8), turned to -90 degrees
- moved C4 15.7 mm to (114.2, 68.0), turned to -90 degrees
- moved C8 15.7 mm to (123.8, 71.4), turned to -90 degrees
- moved R2 13.7 mm to (120.5, 57.1)
- moved R1 13.7 mm to (118.5, 57.1)
- moved R5 13.0 mm to (124.2, 42.0)
- moved SW1 11.1 mm to (113.8, 45.3), turned to 90 degrees
- moved R7 11.1 mm to (122.8, 53.8), turned to 90 degrees
- moved C6 10.0 mm to (122.2, 67.6), turned to -90 degrees
- moved C12 9.72 mm to (120.9, 81.1), turned to 90 degrees
- moved C15 8.63 mm to (116.6, 50.3)
- moved C1 5.76 mm to (121.4, 74.2)
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Connections:
- C12 pad 2: XOUT -> Net-(C12-Pad2)
- C9 pad 1: +3V3 -> Net-(C9-Pad1)
- P3 pad 4: 24 -> 23
- P3 pad 6: +3V3 -> ADC_VREF
- R6 pad 1: QSPI_SS -> XOUT
- R6 pad 2: +3V3 -> Net-(C12-Pad2)
- U1 pad 24: unconnected-(U1-Pad24) -> Net-(J2-Pad1)
- U1 pad 25: unconnected-(U1-Pad25) -> Net-(J2-Pad3)
- U1 pad 35: unconnected-(U1-Pad35) -> 23
- U1 pad 36: 24 -> unconnected-(U1-Pad36)
- U1 pad 43: +3V3 -> Net-(C9-Pad1)
- Y1 pad 3: XOUT -> Net-(C12-Pad2)
Routing:
- net GND: track 105.8 -> 16.2 mm, vias 13 -> 17
- net 24: track 33.9 -> 0.00 mm, vias 1 -> 0
- net 23: track 0.00 -> 31.4 mm, vias 0 -> 1
- net Net-(C9-Pad1): track 0.00 -> 31.4 mm, vias 0 -> 3
- net USB_DM: track 9.56 -> 24.6 mm, vias 2 -> 1
- net Net-(R1-Pad1): track 22.3 -> 7.41 mm, vias 2 -> 1
- net Net-(R2-Pad1): track 21.7 -> 7.59 mm, vias 2 -> 1
- net QSPI_SD3: track 23.9 -> 11.1 mm, vias 2 -> 0
- net +1V1: track 32.4 -> 20.1 mm, vias 0 -> 5
- net Net-(J2-Pad1): track 0.00 -> 11.7 mm
- net USB_DP: track 11.0 -> 22.6 mm, vias 0 -> 2
- net XOUT: track 14.8 -> 3.17 mm
- net ~{RESET}: track 25.7 -> 36.9 mm
- net QSPI_CLK: track 19.7 -> 9.58 mm
- net QSPI_SD0: track 15.4 -> 7.44 mm
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- added copper zone on F.Cu, net +1V1
- added copper zone on F.Cu, net +3V3
- added copper zone on F.Cu, net 17
- added copper zone on F.Cu, net 5
- added copper zone on F.Cu, net XIN
Other:
- board size 21.3 x 51.6 mm -> 20.8 x 51.6 mm
- board text added: "0"
- board text added: "1"
- board text added: "10"
- board text added: "11"
- board text added: "12"
- board text added: "13"
- board text added: "14"
- board text added: "15"
- board text added: "16"
- board text added: "17"
- board text added: "18"
- board text added: "19"
- board text added: "2"
- board text added: "20"
- board text added: "21"
- board text added: "23"
- board text added: "26"
- board text added: "27"
- board text added: "28"
- board text added: "3"
- board text added: "4"
- board text added: "5"
- board text added: "6"
- board text added: "7"
- board text added: "8"
- board text added: "9"
- board text added: "@74th"
- board text added: "A0 26"
- board text added: "A1 27"
- board text added: "A3 28"
- board text added: "RP2040L"
- board text added: "RX"
- board text added: "SCL"
- board text added: "SDA"
- board text added: "SWCK"
- board text added: "SWD"
- board text added: "TX"
- board text added: "TX19 SCK18 CSn17 RX16"
- board text added: "VREF"
- board text added: "v1.4.0"
- board text removed: "16/S0RX I0SDA/U0TX"
- board text removed: "17/S0CSn I0SCL/U0RX"
- board text removed: "18/S0SCK I1SDA"
- board text removed: "19/S0TX I1SCL"
- board text removed: "20/I0SDA"
- board text removed: "21/I0SCL"
- board text removed: "26/ADC0 I1SDA"
- board text removed: "27/ADC1 I1SCL"
- board text removed: "28/ADC2"
- board text removed: "EN"
- board text removed: "RP2040Large"
- board text removed: "S0CSn/1 I0SCL/U0RX"
- board text removed: "S0CSn/5 I0SCL/U1RX"
- board text removed: "S0RX/0 I0SDA/U0TX"
- board text removed: "S0RX/4 I0SDA/U1TX"
- board text removed: "S0SCK/2 I1SDA"
- board text removed: "S0SCK/6 I1SDA"
- board text removed: "S0TX/3 I1SCL"
- board text removed: "S0TX/7 I1SCL"
- board text removed: "S1CSn/13 I0SCL/U0RX"
- board text removed: "S1CSn/9 I0SCL/U1RX"
- board text removed: "S1RX/12 I0SDA/U0TX"
- board text removed: "S1RX/8 I0SDA/U1TX"
- board text removed: "S1SCK/10 I1SDA"
- board text removed: "S1SCK/14 I1SDA"
- board text removed: "S1TX/11 I1SCL"
- board text removed: "S1TX/15 I1SCL"
- board text removed: "v1.0.2"

Commit message: rp2040-large/1.5.0
Parts:
- removed J2: SWD, rp2040-dev-board:SWD_PIN
- removed P3: 20Pin, rp2040-dev-board:SC0915-LIKE
- added CH2: SWD, 74th:PinOut_SWD_3Pin, F.Cu at (147.3, 81.3)
- added D1: RED, 74th:LED_0805_2012, F.Cu at (142.6, 49.7)
- added D2: BLUE, 74th:LED_0805_2012, F.Cu at (144.7, 49.7)
- added MISC-ACCOUNTTEXT: Logo_74th_text, 74th:Logo_74th_text, B.Cu at (139.2, 50.0)
- added MISC-ICON: LOGO, 74th:Logo_74th_5mm, B.Cu at (137.9, 47.1)
- added R6: 10k, 74th:Register_0805_2012, B.Cu at (146.2, 48.7)
- added REF**: JLCJLCJLCJLC, 74th:Logo_JLCJLCJLCJLC, B.Cu at (140.8, 81.8)
- added U1: CH213K, 74th:Package_SOT-23, F.Cu at (140.3, 45.3)
- C1: renamed from C14; footprint rp2040-dev-board:Capacitor_0805_2012 -> 74th:Capacitor_0805_2012
- C10: renamed from C3; footprint rp2040-dev-board:Capacitor_0805_2012 -> 74th:Capacitor_0805_2012
- C11: renamed from C16; footprint rp2040-dev-board:Capacitor_0805_2012 -> 74th:Capacitor_0805_2012
- C12: renamed from C7; footprint rp2040-dev-board:Capacitor_0805_2012 -> 74th:Capacitor_0805_2012
- C13: renamed from C10; footprint rp2040-dev-board:Capacitor_0805_2012 -> 74th:Capacitor_0805_2012
- C14: renamed from C6; footprint rp2040-dev-board:Capacitor_0805_2012 -> 74th:Capacitor_0805_2012
- C15: renamed from C8; footprint rp2040-dev-board:Capacitor_0805_2012 -> 74th:Capacitor_0805_2012
- C16: renamed from C1; footprint rp2040-dev-board:Capacitor_0805_2012 -> 74th:Capacitor_0805_2012
- C2: renamed from C11; footprint rp2040-dev-board:Capacitor_0805_2012 -> 74th:Capacitor_0805_2012
- C3: renamed from C12; footprint rp2040-dev-board:Capacitor_0805_2012 -> 74th:Capacitor_0805_2012
- C4: renamed from C15; footprint rp2040-dev-board:Capacitor_0805_2012 -> 74th:Capacitor_0805_2012
- C5: renamed from C9; footprint rp2040-dev-board:Capacitor_0805_2012 -> 74th:Capacitor_0805_2012
- C6: renamed from C13; footprint rp2040-dev-board:Capacitor_0805_2012 -> 74th:Capacitor_0805_2012
- C7: renamed from C5; footprint rp2040-dev-board:Capacitor_0805_2012 -> 74th:Capacitor_0805_2012
- C8: renamed from C2; footprint rp2040-dev-board:Capacitor_0805_2012 -> 74th:Capacitor_0805_2012
- C9: renamed from C4; footprint rp2040-dev-board:Capacitor_0805_2012 -> 74th:Capacitor_0805_2012
- CH1: renamed from P2; value 20Pin -> RasperryPiPico PinOut; footprint rp2040-dev-board:SC0915-LIKE -> 74th:PinOut_RaspberryPiPico
- J1: value USB2.0_C_v3 -> 217179-0001; footprint rp2040-dev-board:USB-C-12-Pin-MidMount-ali-v4 -> 74th:Connector_USB-C-Receptacle_SMT_12-Pin_MidMount_Simple
- R1: renamed from R6; footprint rp2040-dev-board:Register_0805_2012 -> 74th:Register_0805_2012
- R10: renamed from R8; footprint rp2040-dev-board:Register_0805_2012 -> 74th:Register_0805_2012
- R11: renamed from R3; footprint rp2040-dev-board:Register_0805_2012 -> 74th:Register_0805_2012
- R2: renamed from R5; footprint rp2040-dev-board:Register_0805_2012 -> 74th:Register_0805_2012
- R3: renamed from R4; footprint rp2040-dev-board:Register_0805_2012 -> 74th:Register_0805_2012
- R4: renamed from R1; footprint rp2040-dev-board:Register_0805_2012 -> 74th:Register_0805_2012
- R5: renamed from R2; footprint rp2040-dev-board:Register_0805_2012 -> 74th:Register_0805_2012
- R7: value 1kR -> 5.1k; footprint rp2040-dev-board:Register_0805_2012 -> 74th:Register_0805_2012
- R8: renamed from R10; footprint rp2040-dev-board:Register_0805_2012 -> 74th:Register_0805_2012
- R9: footprint rp2040-dev-board:Register_0805_2012 -> 74th:Register_0805_2012
- SW1, SW2: footprint rp2040-dev-board:SKRPABE010 -> 74th:PushButton_SKRPABE010
- U2: renamed from U3; footprint Package_TO_SOT_SMD:SOT-223-3_TabPin2 -> 74th:Package_SOT-89-3
- U3: renamed from U2; value W25Q128JVS -> W25Q32JVS; footprint rp2040-dev-board:W25Q16-128JV-SOIC -> 74th:Package_SOIC-8_5.23x5.23mm_P1.27mm
- U4: renamed from U1; footprint rp2040-dev-board:RP2040_hand -> 74th:Package_QFN-54-1EP_7x7mm_P0.4mm_EP3.1x3.1mm_hand
- Y1: footprint rp2040-dev-board:Crystal_SMD_3225-4Pin_3.2x2.5mm_HandSoldering -> 74th:Crystal_SMD_3225-4Pin_3.2x2.5mm_HandSoldering
- moved CH1 32.2 mm to (141.0, 43.2)
- moved C7 29.2 mm to (145.3, 61.9), turned to 90 degrees
- moved R11 27.4 mm to (138.7, 59.6), turned to 180 degrees
- moved R4 26.9 mm to (142.8, 45.6), turned to -90 degrees
- moved C1 26.7 mm to (144.1, 45.3), turned to 0 degrees
- moved R10 26.5 mm to (138.7, 57.6), turned to 0 degrees
- moved SW1 25.7 mm to (137.9, 54.4), turned to 0 degrees
- moved C9 24.8 mm to (138.8, 64.6), turned to 180 degrees
- moved C2 24.4 mm to (137.4, 80.0)
- moved R1 24.1 mm to (142.2, 76.8), turned to 0 degrees
- moved C13 24.1 mm to (137.1, 71.5)
- moved Y1 24.1 mm to (141.0, 80.0)
- moved R8 24.1 mm to (146.0, 52.5), turned to -90 degrees
- moved J1 23.9 mm to (141.0, 31.8)
- moved C3 23.6 mm to (144.5, 80.0)
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Connections:
- net 0 renamed /GPIO0
- net 1 renamed /GPIO1
- net 10 renamed /GPIO10
- net 11 renamed /GPIO11
- net 12 renamed /GPIO12
- net 13 renamed /GPIO13
- net 14 renamed /GPIO14
- net 15 renamed /GPIO15
- net 2 renamed /GPIO2
- net 3 renamed /GPIO3
- net 4 renamed /GPIO4
- net 5 renamed /GPIO5
- net 6 renamed /GPIO6
- net 7 renamed /GPIO7
- net 8 renamed /GPIO8
- net 9 renamed /GPIO9
- net Net-(R3-Pad1) renamed /BOOTSEL
- net QSPI_CLK renamed /QSPI_CLK
- net QSPI_SD0 renamed /QSPI_SD0
- net QSPI_SD1 renamed /QSPI_SD1
- net QSPI_SD2 renamed /QSPI_SD2
- net QSPI_SD3 renamed /QSPI_SD3
- net QSPI_SS renamed /QSPI_SS
- net XIN renamed /XIN
- net XOUT renamed /XOUT
- J1 pad 1: +5V -> VBUS
- J1 pad 2: USB_DM -> Net-(J1-D-)
- J1 pad 3: USB_DP -> Net-(J1-D+)
- R4 pad 1: Net-(R1-Pad1) -> Net-(J1-D-)
- R4 pad 2: USB_DP -> /USB_DM
- R5 pad 1: Net-(R2-Pad1) -> Net-(J1-D+)
- R5 pad 2: USB_DM -> /USB_DP
- R7 pad 1: ~{RESET} -> Net-(D1-A)
- R8 pad 2: ADC_VREF -> /ADC_VREF
- R9 pad 1: ADC_VREF -> /ADC_VREF
- SW2 pad 2: ~{RESET} -> /RUN
- U4 pad 24: Net-(J2-Pad1) -> /SWCLK
- U4 pad 25: Net-(J2-Pad3) -> /SWDIO
- U4 pad 26: ~{RESET} -> /RUN
- U4 pad 27: 16 -> /GPIO16
- U4 pad 28: 17 -> /GPIO17
- U4 pad 29: 18 -> /GPIO18
- U4 pad 30: 19 -> /GPIO19
- U4 pad 31: 20 -> /GPIO20
- U4 pad 32: 21 -> /GPIO21
- U4 pad 34: 22 -> /GPIO22
- U4 pad 35: 23 -> unconnected-(U4-GPIO23-Pad35)
- U4 pad 37: unconnected-(U1-Pad37) -> Net-(U4-GPIO25)
- U4 pad 38: 26 -> /GPIO26
- U4 pad 39: 27 -> /GPIO27
- U4 pad 40: 28 -> /GPIO28
- U4 pad 46: Net-(R2-Pad1) -> /USB_DM
- U4 pad 47: Net-(R1-Pad1) -> /USB_DP
Routing:
- net ~{RESET}: track 36.9 -> 0.00 mm, vias 2 -> 0
- net /RUN: track 0.00 -> 32.6 mm, vias 0 -> 3
- net 23: track 31.4 -> 0.00 mm, vias 1 -> 0
- net VBUS: track 0.00 -> 26.9 mm
- net Net-(U4-GPIO25): track 0.00 -> 25.1 mm, vias 0 -> 1
- net USB_DM: track 24.6 -> 0.00 mm, vias 1 -> 0
- net USB_DP: track 22.6 -> 0.00 mm, vias 2 -> 0
- net 28: track 22.5 -> 0.00 mm, vias 1 -> 0
- net /GPIO28: track 0.00 -> 22.0 mm
- net +3V3: track 109.2 -> 90.4 mm, vias 12 -> 16
- net /USB_DP: track 0.00 -> 18.7 mm, vias 0 -> 1
- net /USB_DM: track 0.00 -> 18.6 mm, vias 0 -> 1
- net 27: track 17.2 -> 0.00 mm, vias 1 -> 0
- net /GPIO27: track 0.00 -> 16.6 mm, vias 0 -> 1
- net 26: track 15.8 -> 0.00 mm, vias 1 -> 0
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- removed copper zone on F.Cu, net +1V1
- removed copper zone on F.Cu, net /GPIO5
- removed copper zone on F.Cu, net /XIN
- removed copper zone on F.Cu, net 17
Other:
- board size 20.8 x 51.6 mm -> 20.3 x 50.8 mm
- board text added: "26A0"
- board text added: "27A1"
- board text added: "28A2"
- board text added: "AGND"
- board text added: "CK"
- board text added: "CSn"
- board text added: "DIO"
- board text added: "RP2040-Large"
- board text added: "SCK"
- board text added: "SPITX"
- board text added: "VB US"
- board text added: "v1.5.0"
- board text removed: "23"
- board text removed: "@74th"
- board text removed: "A0 26"
- board text removed: "A1 27"
- board text removed: "A3 28"
- board text removed: "BOOT"
- board text removed: "RP2040L"
- board text removed: "SWCK"
- board text removed: "SWD"
- board text removed: "TX19 SCK18 CSn17 RX16"
- board text removed: "v1.4.0"

Commit message: rp2040-large/1.5.1
Parts:
- moved D2 0.72 mm to (145.4, 49.7)
- moved D1 0.58 mm to (143.2, 49.7)
- moved SW1 0.46 mm to (137.4, 54.4)
- moved SW2 0.33 mm to (144.8, 54.5)
Routing:
- net /RUN: track 32.6 -> 31.8 mm
- net /QSPI_SS: track 14.9 -> 14.2 mm
- net Net-(C3-Pad2): track 4.29 -> 3.63 mm
- net /GPIO28: track 22.0 -> 21.4 mm
- net /GPIO21: track 8.08 -> 7.51 mm
- net /GPIO1: track 33.6 -> 33.0 mm
- net /LED: track 2.75 -> 3.30 mm
- net /GPIO17: track 10.6 -> 10.1 mm
- net /GPIO20: track 6.13 -> 5.60 mm
- net /QSPI_SD3: track 10.7 -> 10.2 mm
- net /QSPI_CLK: track 9.04 -> 8.54 mm
- net /GPIO19: track 5.28 -> 4.78 mm
Other:
- board text added: "25"
- board text added: "A2"
- board text added: "AG"
- board text added: "DCL"
- board text added: "PWR"
- board text added: "RP2040L"
- board text added: "US"
- board text added: "VB"
- board text added: "v1.5.1"
- board text removed: "28A2"
- board text removed: "AGND"
- board text removed: "RP2040-Large"
- board text removed: "VB US"
- board text removed: "v1.5.0"

Commit message: 1.5.2
Other:
- board text added: "v1.5.2"
- board text removed: "v1.5.1"
