File: rp2040-large/rp2040-large.kicad_sch (KiCad schematic)
At the start: 30 parts, among them P1 USB2.0_C_12pin, P2 20Pin, P3 20Pin, SW1 SW_Push, U1 RP2040, U2 W25Q128JVS, U3 AZ1117-3.3, Y1 Crystal_GND24

Commit message: rp2040-large v1.4.0
Parts:
- removed P1: USB2.0_C_12pin, rp2040-dev-board:USB-C-12-Pin-MidMount-ali-v2, symbol rp2040-dev-board:USB2.0_C_12pin
- added C16: 100nF, rp2040-dev-board:Capacitor_0805_2012, symbol Device:C
- added J1: USB2.0_C_v3, rp2040-dev-board:USB-C-12-Pin-MidMount-ali-v4, symbol rp2040-dev-board:USB2.0_C_v3
- added J2: SWD, rp2040-dev-board:SWD_PIN, symbol rp2040-dev-board:SWD
- added R10: 1R, rp2040-dev-board:Register_0805_2012, symbol Device:R
- added R8: 10kR, rp2040-dev-board:Register_0805_2012, symbol Device:R
- added R9: 200R, rp2040-dev-board:Register_0805_2012, symbol Device:R
- added SW2: SW_Push, rp2040-dev-board:SKRPABE010, symbol Switch:SW_Push
- C11, C12: footprint rp2040-dev-board:Capacitor_0603_1608 -> rp2040-dev-board:Capacitor_0805_2012
- C9: value 100nF -> 1uF
- R6: value 10kR -> 1kR
- SW1: footprint rp2040-dev-board:2Pin -> rp2040-dev-board:SKRPABE010
Connections:
- net +3V3: now also C16.1, R8.2, R9.2; no longer C9.1, P3.6, R6.2, U1.43 (ADC_AVDD)
- net +5V: now also J1.1 (VBUS)
- net GND: now also C16.2, J1.4 (GND), J2.2 (GND), SW2.1
- net QSPI_SS: now also R8.1; no longer R6.1
- net USB_DM: now also J1.2 (D-)
- net USB_DP: now also J1.3 (D+)
- net XOUT: now also R6.1; no longer C12.2, Y1.3
- net ~{RESET}: now also SW2.2
- net at R5.1: now also J1.5 (CC1)
- net at R4.1: now also J1.6 (CC2)
- net at U1.24 (SWCLK): now also J2.1 (SWCLK)
- net at U1.25 (SWD): now also J2.3 (SWDIO)
- net 23: now reaches U1.35 (GPIO23)
- net 23: now also P3.4
- net 24: no longer names the net of U1.36 (GPIO24)
- net 24: no longer P3.4
- new net: C12.2, R6.2, Y1.3
- new net: C9.1, R10.1, U1.43 (ADC_AVDD)
- new net ADC_VREF: P3.6, R10.2, R9.1
- no-connect marks 7 -> 3
Other:
- title: (none) -> RP2040-Large-Board
- moved on the sheet: C10, C11, C12, C14, C15, C4, C5, C6, C7, C8, U3, Y1

Commit message: rp2040-large/1.5.0
Parts:
- removed J2: SWD, rp2040-dev-board:SWD_PIN, symbol rp2040-dev-board:SWD
- removed P3: 20Pin, rp2040-dev-board:SC0915-LIKE, symbol rp2040-dev-board:20Pin
- added CH2: SWD, 74th:PinOut_SWD_3Pin, symbol 74th_Interface:SWD_3Pin
- added D1: RED, 74th:LED_0805_2012, symbol Device:LED
- added D2: BLUE, 74th:LED_0805_2012, symbol Device:LED
- added R6: 10k, 74th:Register_0805_2012, symbol Device:R
- added U1: CH213K, 74th:Package_SOT-23, symbol 74th_Passive:CH213K_Ideal-Diode-for-USB-Power
- C1: renamed from C14; footprint rp2040-dev-board:Capacitor_0805_2012 -> 74th:Capacitor_0805_2012
- C10: renamed from C3; footprint rp2040-dev-board:Capacitor_0805_2012 -> 74th:Capacitor_0805_2012
- C11: renamed from C16; footprint rp2040-dev-board:Capacitor_0805_2012 -> 74th:Capacitor_0805_2012
- C12: renamed from C7; footprint rp2040-dev-board:Capacitor_0805_2012 -> 74th:Capacitor_0805_2012
- C13: renamed from C10; footprint rp2040-dev-board:Capacitor_0805_2012 -> 74th:Capacitor_0805_2012
- C14: renamed from C6; footprint rp2040-dev-board:Capacitor_0805_2012 -> 74th:Capacitor_0805_2012
- C15: renamed from C8; footprint rp2040-dev-board:Capacitor_0805_2012 -> 74th:Capacitor_0805_2012
- C16: renamed from C1; footprint rp2040-dev-board:Capacitor_0805_2012 -> 74th:Capacitor_0805_2012
- C2: renamed from C11; footprint rp2040-dev-board:Capacitor_0805_2012 -> 74th:Capacitor_0805_2012
- C3: renamed from C12; footprint rp2040-dev-board:Capacitor_0805_2012 -> 74th:Capacitor_0805_2012
- C4: renamed from C15; footprint rp2040-dev-board:Capacitor_0805_2012 -> 74th:Capacitor_0805_2012
- C5: renamed from C9; footprint rp2040-dev-board:Capacitor_0805_2012 -> 74th:Capacitor_0805_2012
- C6: renamed from C13; footprint rp2040-dev-board:Capacitor_0805_2012 -> 74th:Capacitor_0805_2012
- C7: renamed from C5; footprint rp2040-dev-board:Capacitor_0805_2012 -> 74th:Capacitor_0805_2012
- C8: renamed from C2; footprint rp2040-dev-board:Capacitor_0805_2012 -> 74th:Capacitor_0805_2012
- C9: renamed from C4; footprint rp2040-dev-board:Capacitor_0805_2012 -> 74th:Capacitor_0805_2012
- CH1: renamed from P2; value 20Pin -> RasperryPiPico PinOut; footprint rp2040-dev-board:SC0915-LIKE -> 74th:PinOut_RaspberryPiPico; symbol rp2040-dev-board:20Pin -> 74th_Interface:RaspberryPiPico_PinOut
- J1: value USB2.0_C_v3 -> 217179-0001; footprint rp2040-dev-board:USB-C-12-Pin-MidMount-ali-v4 -> 74th:Connector_USB-C-Receptacle_SMT_12-Pin_MidMount_Simple; symbol rp2040-dev-board:USB2.0_C_v3 -> 74th_Interface:USB_TypeC-2.0_Receptacle
- R1: renamed from R6; footprint rp2040-dev-board:Register_0805_2012 -> 74th:Register_0805_2012
- R10: renamed from R8; footprint rp2040-dev-board:Register_0805_2012 -> 74th:Register_0805_2012
- R11: renamed from R3; footprint rp2040-dev-board:Register_0805_2012 -> 74th:Register_0805_2012
- R2: renamed from R5; footprint rp2040-dev-board:Register_0805_2012 -> 74th:Register_0805_2012
- R3: renamed from R4; footprint rp2040-dev-board:Register_0805_2012 -> 74th:Register_0805_2012
- R4: renamed from R1; footprint rp2040-dev-board:Register_0805_2012 -> 74th:Register_0805_2012
- R5: renamed from R2; footprint rp2040-dev-board:Register_0805_2012 -> 74th:Register_0805_2012
- R7: value 1kR -> 5.1k; footprint rp2040-dev-board:Register_0805_2012 -> 74th:Register_0805_2012
- R8: renamed from R10; footprint rp2040-dev-board:Register_0805_2012 -> 74th:Register_0805_2012
- R9: footprint rp2040-dev-board:Register_0805_2012 -> 74th:Register_0805_2012
- SW1: footprint rp2040-dev-board:SKRPABE010 -> 74th:PushButton_SKRPABE010; Function (none) -> BOOT
- SW2: footprint rp2040-dev-board:SKRPABE010 -> 74th:PushButton_SKRPABE010; Function (none) -> RST
- U2: renamed from U3; footprint Package_TO_SOT_SMD:SOT-223-3_TabPin2 -> 74th:Package_SOT-89-3
- U3: renamed from U2; value W25Q128JVS -> W25Q32JVS; footprint rp2040-dev-board:W25Q16-128JV-SOIC -> 74th:Package_SOIC-8_5.23x5.23mm_P1.27mm; symbol Memory_Flash:W25Q128JVS -> 74th_ApplicationIC:W25Q32JVSS-FLASH
- U4: renamed from U1; footprint rp2040-dev-board:RP2040_hand -> 74th:Package_QFN-54-1EP_7x7mm_P0.4mm_EP3.1x3.1mm_hand; MPN (none) -> C2040
- Y1: footprint rp2040-dev-board:Crystal_SMD_3225-4Pin_3.2x2.5mm_HandSoldering -> 74th:Crystal_SMD_3225-4Pin_3.2x2.5mm_HandSoldering
Connections:
- net +3V3: now also CH1.36 (3V3)
- net +5V: now also CH1.39 (VSYS), U1.2 (VO-); no longer J1.1 (VBUS)
- net ADC_VREF: now also CH1.35 (VREF)
- net GND: now also CH1.23 (GND), CH1.28 (GND), CH1.33 (GND), CH1.38 (GND), CH2.2 (GND), D1.1 (K), D2.1 (K), U1.1 (GND)
- net USB_DM: now also R4.2, U4.46 (USB_DM); no longer J1.2 (D-), R5.2
- net USB_DP: now also R5.2, U4.47 (USB_DP); no longer J1.3 (D+), R4.2
- net at R4.1: now also J1.2 (D-); no longer U4.47 (USB_DP)
- net at R5.1: now also J1.3 (D+); no longer U4.46 (USB_DM)
- net SWCLK: now reaches U4.24 (SWCLK)
- net SWCLK: now also CH2.1 (SWCLK)
- net SWDIO: now reaches U4.25 (SWD)
- net SWDIO: now also CH2.3 (SWDIO)
- net BOOTSEL: now reaches R11.1, SW1.2
- net at U4.37 (GPIO25): now also R6.1
- net 0 renamed GPIO0
- net 1 renamed GPIO1
- net 10 renamed GPIO10
- net 11 renamed GPIO11
- net 12 renamed GPIO12
- net 13 renamed GPIO13
- net 14 renamed GPIO14
- net 15 renamed GPIO15
- net 16 renamed GPIO16
- net GPIO16: now also CH1.21 (16)
- net 17 renamed GPIO17
- net GPIO17: now also CH1.22 (17)
- net 18 renamed GPIO18
- net GPIO18: now also CH1.24 (18)
- net 19 renamed GPIO19
- net GPIO19: now also CH1.25 (19)
- net 2 renamed GPIO2
- net 20 renamed GPIO20
- net GPIO20: now also CH1.26 (20)
- net 21 renamed GPIO21
- net GPIO21: now also CH1.27 (21)
- net 22 renamed GPIO22
- net GPIO22: now also CH1.29 (22)
- net 23: no longer names the net of U4.35 (GPIO23)
- net 26 renamed GPIO26
- net GPIO26: now also CH1.31 (26)
- net 27 renamed GPIO27
- net GPIO27: now also CH1.32 (27)
- net 28 renamed GPIO28
- net GPIO28: now also CH1.34 (28)
- net 3 renamed GPIO3
- net 4 renamed GPIO4
- net 5 renamed GPIO5
- net 6 renamed GPIO6
- net 7 renamed GPIO7
- net 8 renamed GPIO8
- net 9 renamed GPIO9
- net ~{RESET} renamed RUN
- net RUN: now also CH1.30 (RUN); no longer R7.1
- new net: D1.2 (A), R7.1
- new net LED: D2.2 (A), R6.2
- new net VBUS: CH1.40 (VBUS), J1.1 (VBUS), U1.3 (VI+)
- no-connect marks 3 -> 4
Other:
- note added: "Flash"
- note added: "MCU"
- note added: "Oscillator"
- note added: "PinOut"
- note added: "Power"
- note added: "RESET"
- note added: "USB & Power"
- company: (none) -> 74th
- moved on the sheet: C1, C10, C11, C12, C13, C14, C15, C16, C2, C3, C4, C5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

Commit message: rp2040-large/1.5.1
Parts:
- C1, C4: value 10uF -> 10u
- C10, C5, C7: value 1uF -> 1u
- C11, C12, C13, C14, C15, C16, C6, C8, C9: value 100nF -> 100n
- C2, C3: value 27pF -> 20p
- R1, R11: value 1kR -> 1k
- R10: value 10kR -> 10k
- R2, R3: value 5.1kR -> 5.1k
- R4, R5: value 27.4R -> 27.4
- R9: value 200R -> 200
- U2: value AZ1117-3.3 -> AMS1117-3.3
- Y1: value Crystal_GND24 -> 12M
Other:
- moved on the sheet: CH1, CH2

Commit message: 1.5.2
Parts:
- U4: symbol rp2040-dev-board:RP2040 -> 74th_MCU:RP2040
- Y1: symbol Device:Crystal_GND24 -> 74th_PassiveCommon:Crystal_GND24
Other:
- moved on the sheet: C2, C3, R1
