File: rp2350a-full/rp2350a-full.kicad_sch (KiCad schematic)
At the start: 43 parts, among them J1 USB2.0-C_SMT, J2 SWD_10Pin_MCU-Side, SW1 SKRPABE010, SW2 SKRPABE010, U1 RP2350A, U2 AMS1117, U3 W25Q32JVSS, U4 CH213K, Y1 12M

Commit message: fix
Connections:
- net RESET is gone; now on net RUN: CH1.36 (RST)
Changed lines of the file:
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@@
 		)
 	)
-	(label "RESET"
+	(label "RUN"
 		(at 294.64 185.42 180)
 		(fields_autoplaced yes)
