File: rp2350a-full/rp2350a-full.kicad_sch (KiCad schematic)
At the start: 43 parts, among them J1 USB2.0-C_SMT, J2 SWD_10Pin_MCU-Side, SW1 SKRPABE010, SW2 SKRPABE010, U1 RP2350A, U2 CH213K, U3 AMS1117, U4 W25Q32JVSS, Y1 12M

Commit message: wip
Parts:
- U4: value W25Q32JVSS -> W25Q32JVUU; footprint 74th:Package_SOIC-8_5.23x5.23mm_P1.27mm -> 74th:Package_USON-8_3x4mm_P0.8
Other:
- moved on the sheet: C9, R10, R9, SW1, U4

Commit message: rp2350a-full
Parts:
- L1: symbol Device:L -> 74th_PassiveCommon:L_Directed
Other:
- note added: "Debug Port"
- note added: "Flash"
- note added: "MCU"
- note added: "Pin Out"
- note added: "USB Power"
- company: (none) -> Atsushi Morimoto (@74th)
- title: (none) -> RP2350A-Full
- moved on the sheet: C7, C8, C9, CH1, CH2, D1, J1, J2, R10, R11, R7, R8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
