File: rp2350a-full/rp2350a-full.kicad_pcb (KiCad board)
At the start: 2 copper layers, 20.3 x 48.3 mm, 43 parts, among them J1 USB2.0-C_SMT, J2 SWD_10Pin_MCU-Side, SW1 SKRPABE010, SW2 SKRPABE010, U1 RP2350A, U2 AMS1117, U3 W25Q32JVSS, U4 CH213K, Y1 12M

Commit message: fix
Connections:
- CH1 pad 36: /RESET -> /RUN
Routing:
- net /RUN: track 115.8 -> 152.7 mm

Commit message: rp2350-testing/1.0.0
Parts:
- renumbered C20 to C1, C9 to C10, C12 to C11, C6 to C12, C16 to C13, C11 to C15, C7 to C16, C10 to C17, C15 to C18, C8 to C19, C1 to C2, C2 to C4, C18 to C5, C19 to C6, C4 to C7, C5 to C8, C13 to C9, D2 to D1, R8 to R1, R7 to R10, R10 to R11, R9 to R2, R2 to R4, R1 to R5, R11 to R6, R4 to R7, R5 to R8, R6 to R9, U4 to U2, U2 to U3, U3 to U4
Routing:
- net /GPIO12: track 8.78 -> 8.26 mm

Commit message: wip
Parts:
- C18: value 0.1u -> 4.7u
- U4: value W25Q32JVSS -> W25Q32JVUU; footprint 74th:Package_SOIC-8_5.23x5.23mm_P1.27mm -> 74th:Package_USON-8_3x4mm_P0.8
- moved C9 6.43 mm to (69.2, 62.5), turned to 180 degrees
- moved U4 1.10 mm to (68.8, 59.0)
Routing:
- net +3V3: track 82.2 -> 88.8 mm
- net /QSPI_IO2: track 10.8 -> 9.28 mm
- net /QSPI_IO1: track 9.31 -> 8.26 mm
- net /QSPI_SS: track 16.5 -> 17.5 mm
- net /QSPI_IO3: track 8.77 -> 8.03 mm
- net GND: vias 90 -> 87

Commit message: rp2350a-full
Parts:
- added MISC-ACCOUNTTEXT: Logo_74th_text, 74th:Logo_74th_text, B.Cu at (77.9, 58.8)
- added MISC-ICON: LOGO, 74th:Logo_74th_5mm, B.Cu at (76.0, 62.5)
- moved C9 0.40 mm to (69.2, 62.9)
- moved C1 0.24 mm to (77.0, 51.5)
Routing:
- net Net-(U1-ADC_AVDD): track 19.7 -> 21.9 mm
- net +3V3: track 88.8 -> 89.5 mm
