File: rp2350a-testing/rp2350a-testing.kicad_pcb (KiCad board)
At the start: 2 copper layers, 30.5 x 48.3 mm, 46 parts, among them J1 USB2.0-C_SMT, J2 SWD_10Pin_MCU-Side, SW1 SKRPABE010, SW2 SKRPABE010, U1 CH213K, U2 TLV74311, U3 AMS1117, U4 W25Q32JVSS, U5 RP2350A, Y1 12M

Commit message: wip
Parts:
- moved R1 1.30 mm to (79.9, 38.0)
- moved R2 1.30 mm to (79.9, 39.7)
Routing:
- net GND: track 36.4 -> 50.0 mm, vias 224 -> 223
- net /SWDIO: track 66.5 -> 68.4 mm
- net Net-(J1-CC2): track 16.3 -> 15.0 mm
- net Net-(J1-CC1): track 12.8 -> 11.6 mm
- net Net-(U5-VREG_LX): track 6.12 -> 5.50 mm
Other:
- board text added: "5V"
