File: rp2350a-testing/rp2350a-testing.kicad_sch (KiCad schematic)
At the start: 43 parts, among them J1 USB2.0-C_SMT, J2 SWD_10Pin_MCU-Side, SW1 SKRPABE010, SW2 SKRPABE010, U1 RP2350A, U2 CH213K, U3 AMS1117, U4 W25Q32JVSS, Y1 12M

Commit message: rp2350-testing/1.0.0
Parts:
- removed CH1: 18Pin x2, 74th:PinOut_RP2350-Full, symbol 74th_Interface:Pin_19x2_RP2350-Full
- removed U4: W25Q32JVSS, 74th:Package_SOIC-8_5.23x5.23mm_P1.27mm, symbol 74th_ApplicationIC:W25Q32JVSS-FLASH
- added CH1, CH2: Pin_19, 74th:PinOut_Pin_19, symbol 74th_Interface:Pin_19
- added U2: TLV74311, 74th:Package_SOT-23-5, symbol 74th_Passive:TLV74311-Regulator_SOT23-5
- added U4: W25Q32JVSS, 74th:Package_USON-8_3x4mm_P0.8, symbol 74th_ApplicationIC:W25Q32JVUU-FLASH
- C10: footprint 74th:Capacitor_0603_1608 -> 74th:Capacitor_0402_1005
- C11: renamed from C13; footprint 74th:Capacitor_0603_1608 -> 74th:Capacitor_0402_1005
- C12: renamed from C14; footprint 74th:Capacitor_0603_1608 -> 74th:Capacitor_0402_1005
- C13: renamed from C15; footprint 74th:Capacitor_0603_1608 -> 74th:Capacitor_0402_1005
- C14: renamed from C16; footprint 74th:Capacitor_0603_1608 -> 74th:Capacitor_0402_1005
- C15: renamed from C17; footprint 74th:Capacitor_0603_1608 -> 74th:Capacitor_0402_1005
- C16: renamed from C19; footprint 74th:Capacitor_0603_1608 -> 74th:Capacitor_0402_1005
- C17: renamed from C18; value 4.7u -> 0.1u; footprint 74th:Capacitor_0603_1608 -> 74th:Capacitor_0402_1005
- C18: renamed from C5; footprint 74th:Capacitor_0603_1608 -> 74th:Capacitor_0402_1005
- C19: renamed from C6; footprint 74th:Capacitor_0603_1608 -> 74th:Capacitor_0402_1005
- C3: renamed from C9; footprint 74th:Capacitor_0603_1608 -> 74th:Capacitor_0402_1005
- C4: renamed from C12; footprint 74th:Capacitor_0603_1608 -> 74th:Capacitor_0402_1005
- C5: renamed from C3; footprint 74th:Capacitor_0603_1608 -> 74th:Capacitor_0402_1005_m
- C6: renamed from C2; footprint 74th:Capacitor_0603_1608 -> 74th:Capacitor_0402_1005_m
- C8: renamed from C4; footprint 74th:Capacitor_0603_1608 -> 74th:Capacitor_0402_1005_m
- C9: renamed from C11; footprint 74th:Capacitor_0603_1608 -> 74th:Capacitor_0402_1005
- L1: footprint 74th:Inductor_0806_2016 -> 74th:Inductor_4.1x4.5mm_testing
- R10: renamed from R6; footprint 74th:Register_0603_1608 -> 74th:Register_0402_1005
- renumbered C7 to C1, C8 to C2, C1 to C7, CH2 to CH3, R8 to R1, R7 to R2, R1 to R3, R10 to R4, R9 to R5, R3 to R6, R4 to R7, R2 to R8, R5 to R9, U2 to U1, U1 to U5
Connections:
- net +1V1: now also CH2.3, U2.5 (OUT)
- net +3V3: now also CH2.2, U2.1 (IN), U2.3 (EN), U4.8 (VCC)
- net +5V: now also CH2.1
- net ADC_VREF: now also CH2.5
- net GND: now also CH1.19, CH2.19, U2.2 (GND), U4.4 (GND)
- net GPIO0: now also CH1.2
- net GPIO1: now also CH1.3
- net GPIO10: now also CH1.12
- net GPIO11: now also CH1.13
- net GPIO12: now also CH1.14
- net GPIO13: now also CH1.15
- net GPIO14: now also CH1.16
- net GPIO15: now also CH1.17
- net GPIO16: now also CH1.18
- net GPIO17: now also CH2.18
- net GPIO18: now also CH2.17
- net GPIO19: now also CH2.16
- net GPIO2: now also CH1.4
- net GPIO20: now also CH2.15
- net GPIO21: now also CH2.14
- net GPIO22: now also CH2.13
- net GPIO23: now also CH2.12
- net GPIO24: now also CH2.11
- net GPIO25: now also CH2.10
- net GPIO26: now also CH2.9
- net GPIO27: now also CH2.8
- net GPIO28: now also CH2.7
- net GPIO29: now also CH2.6
- net GPIO3: now also CH1.5
- net GPIO4: now also CH1.6
- net GPIO5: now also CH1.7
- net GPIO6: now also CH1.8
- net GPIO7: now also CH1.9
- net GPIO8: now also CH1.10
- net GPIO9: now also CH1.11
- net QSPI_CLK: now also U4.6 (CLK)
- net QSPI_IO0: now also U4.5 (DI(IO0))
- net QSPI_IO1: now also U4.2 (DO(IO1))
- net QSPI_IO2: now also U4.3 (IO2)
- net QSPI_IO3: now also U4.7 (IO3)
- net QSPI_SS: now also U4.1 (~{CS})
- net RUN: now also CH2.4
- net VBUS: now also CH1.1
- net at SW1.2: now also R4.2
- net at SW1.4: no longer R4.2
- net VLEG_LX: no longer names the net of L1.2, U5.48 (VREG_LX)
Other:
- moved on the sheet: C10, C12, C13, C14, C15, C16, C17, C4, C9, D1, J2, R11
